File: LM1205_codex.kicad_sch (KiCad schematic)
At the start: 0 parts

Commit message: Fix LM1205 symbol library
Parts:
- added U1: LM1205, LM1205:LM1205_DIP-28, symbol LM1205:LM1205
Changed lines of the file:
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@@
 (kicad_sch
-	(version 20250114)
-	(generator "eeschema")
-	(generator_version "9.0")
-	(paper "A4")
-	(sheet_instances
-		(path "/"
-			(page "1")
-		)
-	)
-	(embedded_fonts no)
+  (version 20250114)
+  (generator "eeschema")
+  (generator_version "9.0")
+  (paper "A4")
+  (symbol (lib_id "LM1205:LM1205") (at 0 0 0)
+    (unit 1)
+    (in_bom yes) (on_board yes)
+    (property "Reference" "U1" (id 0) (at 0 0 0) (effects (font (size 1.27 1.27))))
+    (property "Value" "LM1205" (id 1) (at 0 -2.54 0) (effects (font (size 1.27 1.27))))
+    (property "Footprint" "LM1205:LM1205_DIP-28" (id 2) (at 0 -5.08 0) (effects (font (size 1.27 1.27))))
+    (property "Datasheet" "" (id 3) (at 0 -7.62 0) (effects (font (size 1.27 1.27)) (hide yes)))
+    (sheetpath (names "/") (tstamps 0))
+  )
+  (sheet_instances
+    (path "/"
+      (page "1")
+    )
+  )
+  (embedded_fonts no)
 )
