File: LM1205_codex.kicad_sch (KiCad schematic)
At the start: 0 parts

Commit message: Fix LM1205 schematic structure
Parts:
- added U1: LM1205, LM1205:LM1205_DIP-28, symbol LM1205:LM1205
Changed lines of the file:
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@@
-(kicad_sch
-	(version 20250114)
-	(generator "eeschema")
-	(generator_version "9.0")
-	(paper "A4")
-	(sheet_instances
-		(path "/"
-			(page "1")
-		)
-	)
-	(embedded_fonts no)
+(kicad_sch (version 20221206) (generator eeschema)
+  (paper "A4")
+  (symbol (lib_id "LM1205:LM1205") (at 0 0 0) (unit 1)
+    (in_bom yes) (on_board yes) (dnp no)
+    (property "Reference" "U1" (at 0 0 0)
+      (effects (font (size 1.27 1.27))))
+    (property "Value" "LM1205" (at 0 -2.54 0)
+      (effects (font (size 1.27 1.27))))
+    (property "Footprint" "LM1205:LM1205_DIP-28" (at 0 -5.08 0)
+      (effects (font (size 1.27 1.27))))
+    (property "Datasheet" "" (at 0 -7.62 0)
+      (effects (font (size 1.27 1.27)) hide))
+    (pin "1")
+    (pin "2")
+    (pin "3")
+    (pin "4")
+    (pin "5")
+    (pin "6")
+    (pin "7")
+    (pin "8")
+    (pin "9")
+    (pin "10")
+    (pin "11")
+    (pin "12")
+    (pin "13")
+    (pin "14")
+    (pin "15")
+    (pin "16")
+    (pin "17")
+    (pin "18")
+    (pin "19")
+    (pin "20")
+    (pin "21")
+    (pin "22")
+    (pin "23")
+    (pin "24")
+    (pin "25")
+    (pin "26")
+    (pin "27")
+    (pin "28")
+    (instances
+      (project "LM1205_codex"
+        (path "/6972ee66-1e52-4fd2-b479-a98194a488ee" (reference "U1") (unit 1))
+      )
+    )
+  )
+  (sheet_instances
+    (path "/" (page "1"))
+  )
 )
